File: emitter.kicad_pcb (KiCad board)
At the start: 2 copper layers, 87 x 57 mm, 21 parts, among them J1 Screw_Terminal_01x02, J2 Screw_Terminal_01x02, Q1 BD436, Q2 BD436, Q3 BD433, Q4 BD433, U1 4049

Commit message: Fixing the schema
Parts:
- added SW1: SW_Push, Button_Switch_THT:SW_PUSH_6mm, F.Cu at (116.0, 123.0)
- Q1, Q2: value BD436 -> BD433
- Q3, Q4: value BD433 -> BD436
- moved Q1 0.54 mm to (123.0, 116.0)
Connections:
- J2 pad 1: +5V -> Net-(J2-Pad1)
- Q1 pad 1: +5V -> Net-(J1-Pad2)
- Q1 pad 2: Net-(J1-Pad2) -> +5V
- Q2 pad 1: +5V -> Net-(J1-Pad1)
- Q2 pad 2: Net-(J1-Pad1) -> +5V
- Q3 pad 1: GND -> Net-(J1-Pad2)
- Q3 pad 2: Net-(J1-Pad2) -> GND
- Q4 pad 1: GND -> Net-(J1-Pad1)
- Q4 pad 2: Net-(J1-Pad1) -> GND
Routing:
- net Net-(J2-Pad1): track 0.00 -> 24.7 mm
- net +5V: track 68.2 -> 59.6 mm
- net GND: track 55.7 -> 58.1 mm
- net Net-(J1-Pad2): track 49.6 -> 50.4 mm
